Commit message: rewrite the ur10 robot urdf

File: Load_URDF_robot/URDF example/ur_description/urdf/ur10_robot.urdf (robot description, URDF)
Before this commit: robot UR10_urdf, 7 links, 6 joints
Joints:
- joint joint1: origin xyz=0.000097 0.013831 0.107586 rpy=-3.141593 3.141593 -3.141593 -> xyz=0.000097 0.013831 0.107586 rpy=-3.14 3.14 0
- joint joint2: origin xyz=-0.000302 0.169547 0.300694 rpy=-3.141593 3.141593 -3.141593 -> xyz=0.000207 -0.000138 -0.000448 rpy=1.571242 0 0
- joint joint3: origin xyz=0.000323 -0.130180 0.591802 rpy=-3.141593 3.141593 -3.141593 -> xyz=0.000323 0.610802 0.130180 rpy=0 0 0
- joint joint4: origin xyz=-0.000271 0.115196 0.295091 rpy=-3.141593 3.141593 -3.141593 -> xyz=0.0000255 0.5759 -0.069749 rpy=0 0 0
- joint joint5: origin xyz=0.000255 0.006251 0.109749 rpy=-3.141593 3.141593 -3.141593 -> xyz=0.000 0.00 0.1 rpy=-1.57 0 0
- joint joint6: origin xyz=-0.000170 0.071019 0.004261 rpy=1.571242 1.677095 0.000447 -> xyz=0 -0.07 0.105 rpy=1.571242 0 0.000
