Commit message: update urdf for ur3 and ur10 robot

File: Load_URDF_robot/URDF example/ur_description/urdf/ur3_robot.urdf (robot description, URDF)
Before this commit: robot UR3__36__, 7 links, 6 joints
Links:
- removed link UR3__36__
- removed link link__39__
- removed link link__42__
- removed link link__45__
- removed link link__48__
- removed link link__51__
- removed link link__54__
- added link base, mass 1.0; collision mesh filename=package://ur_description/meshes/ur3/ur3_base.dae; visual mesh filename=package://ur_description/meshes/ur3/ur3_base_visual.dae
- added link link_1, mass 1.0; collision mesh filename=package://ur_description/meshes/ur3/ur3_link1.dae; visual mesh filename=package://ur_description/meshes/ur3/ur3_link1_visual.dae
- added link link_2, mass 2.5; collision mesh filename=package://ur_description/meshes/ur3/ur3_link2.dae; visual mesh filename=package://ur_description/meshes/ur3/ur3_link2_visual.dae
- added link link_3, mass 2.5; collision mesh filename=package://ur_description/meshes/ur3/ur3_link3.dae; visual mesh filename=package://ur_description/meshes/ur3/ur3_link3_visual.dae
- added link link_4, mass 1.0; collision mesh filename=package://ur_description/meshes/ur3/ur3_link4.dae; visual mesh filename=package://ur_description/meshes/ur3/ur3_link4_visual.dae
- added link link_5, mass 1.0; collision mesh filename=package://ur_description/meshes/ur3/ur3_link5.dae; visual mesh filename=package://ur_description/meshes/ur3/ur3_link5_visual.dae
- added link link_6, mass 1.0; collision cylinder length=0.032068222761154 radius=0.03120630979538; visual mesh filename=package://ur_description/meshes/ur3/ur3_link6_visual.dae
Joints:
- removed joint joint__38__
- added joint joint_1: type revolute, parent base, child link_1, origin xyz=-0.003618 -0.000070 0.104020 rpy=-3.141593 3.141593 -3.141593, axis 0 0 1, limit lower=-6.2831854820251 upper=6.2831854820251 effort=50.0 velocity=3.1415927410126
- joint joint__41__: child link__42__ -> link_2; parent link__39__ -> link_1
- joint joint__44__: child link__45__ -> link_3; parent link__42__ -> link_2
- joint joint__47__: child link__48__ -> link_4; parent link__45__ -> link_3
- joint joint__50__: child link__51__ -> link_5; parent link__48__ -> link_4
- joint joint__53__: child link__54__ -> link_6; parent link__51__ -> link_5

Commit message: rewrite ur3 robot urdf

File: Load_URDF_robot/URDF example/ur_description/urdf/ur3_robot.urdf (robot description, URDF)
Before this commit: robot UR3_urdf, 7 links, 6 joints
Joints:
- removed joint joint__41__
- removed joint joint__44__
- removed joint joint__47__
- removed joint joint__50__
- removed joint joint__53__
- added joint joint_2: type revolute, parent link_1, child link_2, origin xyz=0 0.05 0.0055 rpy=1.57 3.141593 -3.141593, axis 0 0 1, limit lower=-6.2831854820251 upper=6.2831854820251 effort=50.0 velocity=3.1415927410126
- added joint joint_3: type revolute, parent link_2, child link_3, origin xyz=0 -0.245 0 rpy=0 0 -3.141593, axis 0 0 1, limit lower=-6.2831854820251 upper=6.2831854820251 effort=50.0 velocity=3.1415927410126
- added joint joint_4: type revolute, parent link_3, child link_4, origin xyz=0 0.211 0.00 rpy=-3.141593 3.141593 -3.141593, axis 0 0 1, limit lower=-6.2831854820251 upper=6.2831854820251 effort=50.0 velocity=6.2831854820251
- added joint joint_5: type revolute, parent link_4, child link_5, origin xyz=0 0 0.058 rpy=1.57 3.141593 3.14, axis 0 0 1, limit lower=-6.2831854820251 upper=6.2831854820251 effort=50.0 velocity=6.2831854820251
- added joint joint_6: type continuous, parent link_5, child link_6, origin xyz=0 0 0.0835 rpy=-1.570796 3.141593 -3.14, axis 0 0 1
- joint joint_1: origin xyz=-0.003618 -0.000070 0.104020 rpy=-3.141593 3.141593 -3.141593 -> xyz=-0.003618 -0.000070 0.104020 rpy=-3.14 3.141593 -3.141593

Commit message: update urdf

File: Load_URDF_robot/URDF example/ur_description/urdf/ur3_robot.urdf (robot description, URDF)
Before this commit: robot UR3_urdf, 7 links, 6 joints
Joints:
- joint joint_1: origin xyz=-0.003618 -0.000070 0.104020 rpy=-3.14 3.141593 -3.141593 -> xyz=0 0.004 0.104020 rpy=-3.14 3.141593 -3.141593
